File: HCTL200_2axis.sch (EAGLE design)
At the start: 10 parts, among them IC1 HCTL2000N, IC2 HCTL2000N

Commit message: Add files via upload
Parts:
- removed X1: (no value), con-wago-500:W237-6
- added ANALOG1: (no value), con-lstb:MA04-1
- added C1, C2: (no value), rcl:C-EU025-030X050
- added DIGITAL1, DIGITAL2, POWER1, SERIAL: (no value), con-lstb:MA03-1
- renumbered SV2 to ENC2, SV3 to ENC1
Connections:
- new net N$11: ENC1.4, U$1.D3
- new net N$19: ENC2.4, U$1.D2
- new net N$20: DIGITAL1.2, U$1.D4
- new net N$21: DIGITAL2.2, U$1.D5
- new net N$22: ANALOG1.2, U$1.A6
- new net N$23: ANALOG1.3, U$1.A7
- new net N$28: SERIAL.2, U$1.RX1
- new net N$29: SERIAL.3, U$1.TX0
- net VDD: now also ANALOG1.4, C1.1, C2.1, DIGITAL1.3, DIGITAL2.3, ENC1.1, ENC2.1, POWER1.3
- net VSS: now also ANALOG1.1, C1.2, C2.2, DIGITAL1.1, DIGITAL2.1, ENC1.5, ENC2.5, POWER1.1, U$1.GND2
